File: gauge/gauge.kicad_pcb (KiCad board)
At the start: 2 copper layers, 25 parts, among them J1 PWR, J3 LCD, J4 IO, SW1 NEXT, SW2 PREV, SW3 ENTER, SW4 RESET, U1 ATmega328P-PU, U2 LM1117-5.0, U3 LM1117-5.0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

Commit message: fix schematic
Parts:
- moved D1 1.02 mm to (64.6, 118.5)
Connections:
- D1 pad 4: LED_DIN -> Net-(D1-Pad4)
- D6 pad 2: Net-(D6-Pad2) -> LED_DIN
Routing:
- net LED_DIN: track 108.0 -> 0.00 mm
- net GND: track 203.1 -> 206.4 mm
- net Net-(D1-Pad2): track 7.86 -> 6.84 mm
- added copper zone on F.Cu, net LED_DIN
